File: Hardware/OpenBook_Schematic.sch (EAGLE design)
At the start: 103 parts, among them IC1 BD5229G-TR, IC4 XC6220A331MR-G, J1 FH34SRJ-24S-0.5SH_99_, J2 SAMACSYS_PARTS_USB4110-GF-A, J3 QWIIC_RIGHT_ANGLE, J4 112A-TAAR-R03_ATTEND112ATA, Q1 20V/4.2A/52mΩ/1.4W, Q2 20V/4.2A/52mΩ/1.4W, Q3 SI1308EDL-T1-GE3, U1 W25Q512JVEIQ, U2 ESP32-C6-WROOM-1-N8, U3 DS3231SN#, U4 MAX17048G+T10

Commit message: Changes after review
Signed-off-by: gabrielpitic <gabrielpitic31@gmail.com>
Parts:
- D10: value (none) -> PGB1010603MR; device DeskAssistant v19 v1:EAGLE-LTSPICE_CC0402 -> DeskAssistant v19 v1:PGB1010603MR
- R_BOOT: device DeskAssistant v19 v1:EAGLE-LTSPICE_CC0402 -> DeskAssistant v19 v1:ESP32_WROVER_EAGLE-LTSPICE_RR0402
Other:
- moved on the sheet: EPD_C11, EPD_C7, EPD_C9, R_BOOT
